File: KiCad/authenticator/NHD0420CW_over_SPI.sch (KiCad schematic (older format))
At the start: 2 parts

Commit message: Working with OLED PCB.
Connections:
- net GND: now reaches H4.6 (P6), NHD1.1 (VSS), NHD1.10 (D3), NHD1.11 (D4), NHD1.12 (D5), NHD1.13 (D6), NHD1.14 (D7), NHD1.17 (BS0), NHD1.18 (BS1), NHD1.19 (BS2), NHD1.20 (VSS(Frame)), NHD1.3 (REGVDD), NHD1.4 (D/C), NHD1.5 (R/W), NHD1.6 (E)
- net CS: now reaches H4.2 (P2), NHD1.15 (CS)
- net RES: now reaches H4.1 (P1), NHD1.16 (RES)
- net 3V3: now reaches H4.7 (P7), NHD1.2 (VDD)
- net D0: now reaches H4.5 (P5), NHD1.7 (D0)
- net D1: now reaches H4.4 (P4), NHD1.8 (D1)
- net D2: now reaches H4.3 (P3), NHD1.9 (D2)
Changed lines of the file:
@@
 Connection ~ 4300 4550
 Connection ~ 4300 2650
+Text Label 4450 3050 0    68   ~ 0
+3V3
+Text Label 4450 3150 0    68   ~ 0
+GND
+Text Label 4450 3250 0    68   ~ 0
+D0
+Text Label 4450 3350 0    68   ~ 0
+D1
+Text Label 4450 3450 0    68   ~ 0
+D2
+Text Label 4550 3550 0    68   ~ 0
+CS
+Text Label 4750 3650 2    68   ~ 0
+RES
 $EndSCHEMATC

Commit message: Massive overhaul where ribbon cables are replaced with Cat-cables. New enclosure and button. Various improvements.
Parts:
- H4: symbol HEADER_S_1X07 -> authenticator-rescue:HEADER_S_1X07; Manufacturer (none) -> Molex; Model (none) -> 22-10-2074; Supplier (none) -> www.mouser.fi; Title (none) -> Headers & Wire Housings KK 100 Hdr Flat VERT 20 Au 7Ckt
- NHD1: symbol NHD-0420CW-AB3 -> authenticator-rescue:NHD-0420CW-AB3; Manufacturer (none) -> Newhaven Display; Model (none) -> NHD-0420CW-AY3; Title (none) -> OLED Displays & Accessories 4x20 Yellow Slim Character OLED
Changed lines of the file:
@@
-EESchema Schematic File Version 2
-LIBS:power
-LIBS:device
-LIBS:transistors
-LIBS:conn
-LIBS:linear
-LIBS:regul
-LIBS:74xx
-LIBS:cmos4000
-LIBS:adc-dac
-LIBS:memory
-LIBS:xilinx
-LIBS:microcontrollers
-LIBS:dsp
-LIBS:microchip
-LIBS:analog_switches
-LIBS:motorola
-LIBS:texas
-LIBS:intel
-LIBS:audio
-LIBS:interface
-LIBS:digital-audio
-LIBS:philips
-LIBS:display
-LIBS:cypress
-LIBS:siliconi
-LIBS:opto
-LIBS:atmel
-LIBS:contrib
-LIBS:valves
-LIBS:ds18b20+
-LIBS:ec2-3tnu
-LIBS:at-1220-twt-5v-r
-LIBS:nhd-0420cw-ab3
-LIBS:ec2-nu
-LIBS:headers
-LIBS:Koha-Suomi
+EESchema Schematic File Version 4
 LIBS:authenticator-cache
-EELAYER 25 0
+EELAYER 26 0
 EELAYER END
 $Descr A4 11693 8268
@@
 $EndDescr
 $Comp
-L NHD-0420CW-AB3 NHD1
+L authenticator-rescue:NHD-0420CW-AB3 NHD1
 U 1 1 598B2F34
 P 3800 3250
@@
 F 1 "NHD-0420CW-AB3" H 3600 2400 60  0000 C CNN
 F 2 "Koha-Suomi:Pin_Header_Straight_1x20_Pitch2.54mm" H 3800 3250 60  0001 C CNN
-F 3 "" H 3800 3250 60  0001 C CNN
+F 3 "https://www.mouser.fi/datasheet/2/291/NHD-0420CW-AY3-587980.pdf" H 3800 3250 60  0001 C CNN
+F 4 "NHD-0420CW-AY3" H 3800 3250 50  0001 C CNN "Model"
+F 5 "OLED Displays & Accessories 4x20 Yellow Slim Character OLED" H 3800 3250 50  0001 C CNN "Title"
+F 6 "Newhaven Display" H 3800 3250 50  0001 C CNN "Manufacturer"
 	1    3800 3250
 	0    1    1    0
@@
 OLED display over SPI
 $Comp
-L HEADER_S_1X07 H4
+L authenticator-rescue:HEADER_S_1X07 H4
 U 1 1 598B3472
 P 4950 3200
@@
 F 1 "HEADER_S_1X07" V 5050 3350 50  0000 C CNN
 F 2 "Koha-Suomi:Pin_Header_Straight_1x07_Pitch2.54mm" H 4950 3200 50  0001 C CNN
-F 3 "" H 4950 3200 50  0000 C CNN
+F 3 "https://www.mouser.fi/datasheet/2/276/022102074_sd-589973.pdf" H 4950 3200 50  0001 C CNN
+F 4 "22-10-2074" H 4950 3200 50  0001 C CNN "Model"
+F 5 "www.mouser.fi" H 4950 3200 50  0001 C CNN "Supplier"
+F 6 "Headers & Wire Housings KK 100 Hdr Flat VERT 20 Au 7Ckt" H 4950 3200 50  0001 C CNN "Title"
+F 7 "Molex" H 4950 3200 50  0001 C CNN "Manufacturer"
 	1    4950 3200
 	1    0    0    1
@@
 	2850 4800 5250 4800
 Wire Notes Line
-	2850 2400 4350 2400
-Wire Notes Line
 	5250 2300 2850 2300
 Wire Notes Line
@@
 Wire Notes Line
 	2850 2300 2850 4800
-Wire Notes Line
-	5250 2400 4250 2400
 Wire Wire Line
-	3700 3150 4750 3150
+	3700 3150 4300 3150
 Wire Wire Line
-	4300 2650 4300 4550
+	4300 2650 4300 2850
 Wire Wire Line
 	4300 4550 3700 4550
@@
 	3700 3950 4300 3950
 Connection ~ 4300 3950
-Connection ~ 4300 4550
-Connection ~ 4300 2650
 Text Label 4450 3050 0    68   ~ 0
 3V3
@@
 Text Label 4750 3650 2    68   ~ 0
 RES
+Wire Wire Line
+	4300 3150 4750 3150
+Wire Wire Line
+	4300 3150 4300 3550
+Wire Wire Line
+	4300 2850 4300 2950
+Wire Wire Line
+	4300 2950 4300 3050
+Wire Wire Line
+	4300 3050 4300 3150
+Wire Wire Line
+	4300 3550 4300 3650
+Wire Wire Line
+	4300 3650 4300 3750
+Wire Wire Line
+	4300 4250 4300 4350
+Wire Wire Line
+	4300 4350 4300 4450
+Wire Wire Line
+	4300 4450 4300 4550
+Wire Wire Line
+	4300 3750 4300 3850
+Wire Wire Line
+	4300 3850 4300 3950
+Wire Wire Line
+	4300 3950 4300 4250
+Wire Notes Line
+	2850 2400 5250 2400
 $EndSCHEMATC
