File: KiCad/authenticator/authenticator.kicad_sch (KiCad schematic)
At the start: 94 parts, among them IC1 P82B96P, J1 SS-60300-010, J10 90148-1102, J11 90148-1102, J12 90148-1102, J13 SS-60300-010, J14 SS-60300-010, J2 Screw_Terminal_01x04, J4 694106301002, J5 694106301002, J6 Screw_Terminal_01x03, J7 Screw_Terminal_01x02, J8 90148-1102, J9 90148-1102, T1 Screw_Terminal_01x02, T2 Screw_Terminal_01x02, U1 Wall_PSU_15V, U2 ESP32-S3-DEVKITM-1-N8

Commit message: WIP2
Parts:
- removed BCR1: WGC-300-USB-AT, Koha-Suomi:Bad_board_tag, symbol authenticator-rescue:WGC-300-USB-AT
- removed BJT3, BJT4: KSD471AYTA, Koha-Suomi:KSD471AYTA, symbol authenticator-rescue:KSD471AYTA
- removed D5, D6: D, Koha-Suomi:1N4154TAP, symbol authenticator-rescue:D
- removed EC3: EC2-3TNU, Koha-Suomi:EC2-3TNU, symbol authenticator-rescue:EC2-3TNU
- removed H18, H8: HEADER_S_1X07, Koha-Suomi:Pin_Header_Straight_1x07_Pitch2.54mm, symbol authenticator-rescue:HEADER_S_1X07
- removed J2: Screw_Terminal_01x04, Koha-Suomi:Terminal 1x4 (Molex-398800304), symbol Connector:Screw_Terminal_01x04
- removed J6: Screw_Terminal_01x03, Koha-Suomi:Terminal 1x3 (Molex-398800303), symbol Connector:Screw_Terminal_01x03
- removed J7: Screw_Terminal_01x02, Koha-Suomi:Terminal 1x2 (Molex-398800302), symbol Connector:Screw_Terminal_01x02
- removed R5: 50, Koha-Suomi:Resistor_ThroughHole_6.3x2.3mm_Spacing2.54mm, symbol authenticator-rescue:R
- removed R8, R9: 3.3k, Koha-Suomi:Resistor_ThroughHole_6.3x2.3mm_Spacing2.54mm, symbol Device:R
- removed RPi1: RPi_GPIO, Koha-Suomi:PI_GPIO_Header_F_2x20, symbol authenticator-rescue:RPi_GPIO-Koha-Suomi
- removed US1: USB-Stick, symbol authenticator-rescue:USB-Stick-Koha-Suomi
- removed USBm1: Cable_USB_Micro_m, Koha-Suomi:Bad_board_tag, symbol authenticator-rescue:Cable_USB_Micro_M
- added BCR1: Barcode_Reader Alternate, Koha-Suomi:Bad_board_tag, symbol authenticator-rescue:Barcode_Reader-Koha-Suomi
- added BCR2: Barcode_Reader, Koha-Suomi:RT830C, symbol authenticator-rescue:Barcode_Reader-Koha-Suomi
- added BJT7: BJT NPN, Koha-Suomi:KSD471AYTA, symbol authenticator-rescue:KSD471AYTA
- added H13: HEADER_A_1X05_F, components:38001335, symbol authenticator-rescue:HEADER_A_1X05_F
- added H16: HEADER_A_1X08_F, components:38-00-1338, symbol authenticator-rescue:HEADER_A_1X08_F
- added H17, H8: HEADER_S_1X07_stacking, Koha-Suomi:Pin_Header_Straight_1x07_Pitch2.54mm_stacking, symbol authenticator-rescue:HEADER_S_1X07_stacking
- added H18: HEADER_A_1X02, Koha-Suomi:Pin_Header_Angled_1x02_Pitch2.54mm, symbol authenticator-rescue:HEADER_A_1X02
- added H2: HEADER_A_1X04_F, components:33-00-1334, symbol authenticator-rescue:HEADER_A_1X04_F
- added IC2: Line Driver, components:P82B96P, symbol P82B96P:P82B96P
- added J15, J16: HEADER_S_01x22_low, components:SLW-122-01-X-S, symbol SLW-122-01-T-S:SLW-122-01-T-S
- added J17: HEADER_02x06_F_LOW, components:SLW-106-01-X-D, symbol Connector_Generic:Conn_02x06_Odd_Even
- added J18: HEADER_02x06, components:TSW-106-23-T-D, symbol Connector_Generic:Conn_02x06_Odd_Even
- added J2: HEADER_S_02x20_F_PRT, components:PRT-16763, symbol PRT-16763:PRT-16763
- added J7: FPC breakout, Koha-Suomi:FPC_Breakout_12P_2.54mm, symbol Connector_Generic:Conn_02x06_Odd_Even
- added Q1: RX3L07BGNC16, components:RX3L07BGNC16, symbol RX3L07BGNC16:RX3L07BGNC16
- added R5: 3.3k, Koha-Suomi:Resistor_ThroughHole_Vertical_6.3x2.3mm_Spacing2.54mm, symbol Device:R
- added RFID1: RFID-8P, Koha-Suomi:Bad_board_tag, symbol authenticator-rescue:RFID-8P
- added S1: Push Button, TL2202OAYA, symbol TL2202OAYA:TL2202OAYA
- added SCRLID2, SCRLID3, SCRLID4, SCRLID5, SCRLID6: Screw, Koha-Suomi:Bad_board_tag, symbol authenticator-rescue:Screw
- added SSW1, SSW2, SSW3, SSW4: Screw M3 20mm, Koha-Suomi:Bad_board_tag, symbol authenticator-rescue:Screw
- added STO3, STO4, STO5, STO6, STO7, STO8: Standoff M3 20mm, Koha-Suomi:Standoff M2.5 20x5mm, symbol authenticator-rescue:Standoff-Koha-Suomi
- added THS1: Humid sensor I2C, Koha-Suomi:Bad_board_tag, symbol authenticator-rescue:CC2D33S-SIP
- added U3: Gate Driver, components:MIC4423YN, symbol MIC4423YN:MIC4423YN
- added U4, U5, U6, U7: Nut M3, Koha-Suomi:Bad_board_tag, symbol authenticator-rescue:Nut
- AST1: value AST-1732MR-R -> Piezo; Supplier (none) -> mouser.fi
- BJT1, BJT2, BJT5, BJT6: value KSD471AYTA -> BJT NPN; Supplier Mouser -> mouser.fi
- D1, D2, D4, EC1, EC2, H7, HS1, HS2, T1, T2: Supplier (none) -> mouser.fi
- GROMMETBACK1: renamed from GROMMETBACK; footprint (none) -> Koha-Suomi:Bad_board_tag; Supplier rs.delivers.fi -> fi.rsdelivers.com
- GROMMETSCREW1: renamed from GROMMETSCREW; footprint (none) -> Koha-Suomi:Bad_board_tag; Supplier rs.delivers.fi -> fi.rsdelivers.com
- H1, H15, H4, H9: ALV0%€ 1.52 -> 0.605; Height (none) -> 13.21; Manufacturer Molex -> Samtec; Model 22-10-2074 -> TSW-107-15-T-S; Supplier www.mouser.fi -> mouser.fi; Title Headers & Wire Housings KK 100 Hdr Flat VERT 20 Au 7Ckt -> Headers & Wire Housings Classic PCB Header Strips, 0.100" p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
- H10, H3, H5, H6: Supplier Mouser -> mouser.fi
- H11: footprint (none) -> Koha-Suomi:Pin_Header_Straight_1x20_Pitch2.54mm; ALV0%€ (none) -> 0.552; Height (none) -> 8.74; Manufacturer (none) -> Harwin; Model HEADER M 1x20 -> M20-9992046; Supplier (none) -> mouser.fi
- IC1: value P82B96P -> Line Driver; footprint DIP794W53P254L959H508Q8N -> components:P82B96P; ALV0%€ (none) -> 3.91; Manufacturer (none) -> Texas Instruments; Manufacturer_Name Texas Instruments -> (none); Manufacturer_Part_Number P82B96P -> (none); Model (none) -> P82B96P; Mouser Part Number 595-P82B96P -> (none); Mouser Price/Stock https://www.mouser.co.uk/ProductDetail/Texas-Instruments/P8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 -> (none); Supplier (none) -> mouser.fi; Title (none) -> Buffers & Line Drivers Dual Bidirectional Bus Buffer
- J1, J13, J14: value SS-60300-010 -> Ethernet Socket; footprint SS60300010 -> components:SS60300010; ALV0% 2.46 -> (none); ALV0%€ (none) -> 2.46; Manufacturer (none) -> Bel; Manufacturer_Name Bel -> (none); Manufacturer_Part_Number SS-60300-010 -> (none); Model (none) -> SS-60300-010; Mouser Part Number 530-SS-60300-010 -> (none); Supplier (none) -> mouser.fi; Title (none) -> Modular Connectors / Ethernet Connectors RJ45 Connector
- J10, J11, J12, J8, J9: value 90148-1102 -> HEADER_A_01x02_CGrid; ALV0% 0.911 -> (none); ALV0%€ (none) -> 0.911; Manufacturer (none) -> Molex; Manufacturer_Name Molex -> (none); Manufacturer_Part_Number 90148-1102 -> (none); Model (none) -> 90148-1102; Mouser Part Number 538-90148-1102 -> (none); Mouser Price/Stock https://www.mouser.co.uk/ProductDetail/Molex/90148-1102?qs=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 -> (none); Supplier Mouser -> mouser.fi; Title (none) -> Headers & Wire Housings C-Grid PCB Conn SR H Horz Poly Sn-A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
- J4, J5: value 694106301002 -> Barrel Jack; footprint 694106301002_1 -> components:694106301002_1; ALV0% 0.949 -> (none); ALV0%€ (none) -> 0.949; Manufacturer (none) -> Wurth Elektronik; Manufacturer_Name Wurth Elektronik -> (none); Manufacturer_Part_Number 694106301002 -> (none); Model (none) -> 694106301002; Mouser Part Number 710-694106301002 -> (none); Mouser Price/Stock https://www.mouser.co.uk/ProductDetail/Wurth-Elektronik/694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 -> (none); Supplier (none) -> mouser.fi; Title (none) -> DC Power Connectors WR-DC PwrJk CtrPnTHT Right Angled
- JU1, JU2, JU3, JU4: ALV0% 0.1 -> (none); ALV0%€ (none) -> 0.1
- KP1: footprint Koha-Suomi:Pin_Header_Straight_1x05_Pitch2.54mm -> Koha-Suomi:Bad_board_tag
- LED1: value WP154A4SUREQBFZGC -> RGBLED; footprint Koha-Suomi:WP154A4SUREQBFZGC_real -> Koha-Suomi:WP154A4SUREQBFZGC
- N1, N2, N3: footprint (none) -> Koha-Suomi:Bad_board_tag
- NHD1: value NHD-0420CW-AB3 -> NHD-0420CW-AW3; footprint Koha-Suomi:Pin_Header_Straight_1x20_Pitch2.54mm -> components:NHD0420CWAW3; ALV0%€ 25.06 -> 33.73; Height (none) -> 7; Model NHD-0420CW-AY3 -> NHD-0420CW-AW3; Title OLED Displays & Accessories 4x20 Yellow Slim Character OLED -> (none)
- PS1: footprint NSD1512S5 -> components:NSD1512S5; ALV0% 17.76 -> (none); ALV0%€ (none) -> 17.76; Manufacturer (none) -> Mean Well; Manufacturer_Name Mean Well -> (none); Manufacturer_Part_Number NSD15-12S5 -> (none); Model (none) -> NSD15-12S5; Mouser Part Number 709-NSD15-12S5 -> (none); Mouser Price/Stock https://www.mouser.co.uk/ProductDetail/MEAN-WELL/NSD15-12S5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 -> (none); Supplier (none) -> mouser.fi; Title (none) -> Isolated DC/DC Converters - Through Hole 15W 5V/3A W/EMI FI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
- PS2: footprint SCWN06A05 -> components:SCWN06A05; ALV0% 12.40 -> (none); ALV0%€ (none) -> 12.40; Manufacturer (none) -> Mean Well; Manufacturer_Name Mean Well -> (none); Manufacturer_Part_Number SCWN06A-05 -> (none); Model (none) -> SCWN06A-05; Mouser Part Number 709-SCWN06A-05 -> (none); Mouser Price/Stock https://www.mouser.co.uk/ProductDetail/MEAN-WELL/SCWN06A-05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 -> (none); Supplier Mouser -> mouser.fi; Title (none) -> Isolated DC/DC Converters - Through Hole 6W 9-18Vin 5Vout 1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
- R10, R11, R6, R7: ALV0%€ (none) -> 0.029; Manufacturer (none) -> KOA Speer; Model (none) -> MF1/4DCT52R3301F; Supplier (none) -> mouser.fi; Title (none) -> Metal Film Resistors - Through Hole 1/4 WATT 3.3K OHM 1%
- R4: footprint Koha-Suomi:Resistor_ThroughHole_6.3x2.3mm_Spacing2.54mm -> Koha-Suomi:Resistor_ThroughHole_Vertical_6.3x2.3mm_Spacing2.54mm; Manufacturer KOE Speer -> KOA Speer
- RPE1: ALV0%€ 5.40 -> 2.75; Model ASM-1900036-12_Bulk -> ASM-1900036-22; Title Raspberry Pi 3 Enclosure, White (bulk) -> DesignSpark ABS Case for use with Raspberry Pi 2B, Raspberr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
- SCRLID1: renamed from SCREWLID; footprint (none) -> Koha-Suomi:Bad_board_tag; ALV0%€ 0,78 -> 0.78; Supplier rs.delivers.fi -> fi.rsdelivers.com
- SD1: ALV0%€ 12 -> 16.25; Manufacturer Raspberry Pi -> Kingston; Model NOOBS_32GB_Retail -> SDIT/16GB; Supplier fi.rsdelivers.com -> mouser.fi; Title SD Card preloaded with NOOBS - 32GB -> Memory Cards 16G SDHC Industrial pSLC
- SOC1: footprint Koha-Suomi:Bad_board_tag -> components:RASPBERRY_PI_3_MODEL_B_; symbol authenticator-rescue:SoC-Koha-Suomi -> authenticator-rescue:RPi_GPIO-Koha-Suomi; ALV0%€ 39.30 -> 32.55; Model Raspberry Pi 3 Model B+ -> SC0022; Supplier fi.rsdelivers.com -> mouser.fi; Title Raspberry Pi 3 Model B+ -> Single Board Computers Raspberry Pi 3 Model B V1.2
- STO1, STO2: value Standoff x2 -> Standoff M3 20mm; footprint Koha-Suomi:Bad_board_tag -> Koha-Suomi:Standoff M2.5 20x5mm; ALV0%€ 1.14 -> 0.472; Manufacturer Adafruit -> Keystone Electronics; Model 2337 -> 25505; Supplier thepihut.com -> mouser.fi; Title Adafruit Brass M2.5 Standoffs 16mm tall - Black Plated - Pa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 -> Standoffs & Spacers 5.0 HEX 20.0mm NYLON
- TH1: footprint Koha-Suomi:Bad_board_tag -> Koha-Suomi:HPG-2_08-75X35-12-30
- U2: value ESP32-S3-DEVKITM-1-N8 -> ESP32-S3-DevKitM-1-N8; footprint ESP32-S3-DEVKITM-1-N8:MODULE_ESP32-S3-DEVKITM-1-N8 -> components:MODULE_ESP32-S3-DEVKITM-1-N8; ALV0% 13.95 -> (none); ALV0%€ (none) -> 13.95; Availability In Stock -> (none); Check_prices https://www.snapeda.com/parts/ESP32-S3-DEVKITM-1-N8/Espress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 -> (none); MF Espressif Systems -> (none); MP ESP32-S3-DEVKITM-1-N8 -> (none); Manufacturer_Part_Number ESP32-S3-DevKitM-1-N8 -> (none); Model (none) -> ESP32-S3-DEVKITM-1-N8; PARTREV 1.0 -> (none); Package None -> (none); Price None -> (none); Purchase-URL https://www.snapeda.com/api/url_track_click_mouser/?unipart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 -> (none); STANDARD Manufacturer Recommendations -> (none); SnapEDA_Link https://www.snapeda.com/parts/ESP32-S3-DEVKITM-1-N8/Espress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 -> (none); Supplier Mouser -> mouser.fi
- USBTTL1: ALV0% 20.74 -> (none); ALV0%€ (none) -> 20.74; Manufacturer (none) -> FTDI; Manufacturer_Name FTDI -> (none); Manufacturer_Part_Number TTL-232R-RPI -> (none); Model (none) -> TTL-232R-RPI; Supplier Mouser -> mouser.fi
- ZM1: value ZM10E10B01 -> Snap Switch; ALV0%€ 2.81 -> 1.33; Manufacturer Honeywell -> E-Switch; Model ZM10E10C01 -> MS0850501F025C1A; Title Basic / Snap Action Switches BASIC SW ES -> Basic / Snap Action Switches SPDT 5A OF 25g
Connections:
- net KeyPadPSU+_2 is gone; now on net KeyPadPSU+: H15.1 (P1)
- net RU-5V is gone; now on net R-5V: PS1.7 (-VOUT)
- net B3,4V: now also R2.2, H2.2; no longer H1.3 (P3), LED1.3 (BLUE_CATHODE)
- net D1Close: now also J2.23
- net D1Open: now also J2.21
- net D2Close: now also J2.27
- net D2Open: now also J2.25
- net D3Close: now also J2.35
- net D3Open: now also J2.31
- net D4Close: now also J2.39
- net D4Open: now also J2.37
- net ENCL_DOOR: now also J16.11
- net G3,3V: now also R3.2, H2.1; no longer H1.4 (P4), LED1.4 (GREEN_CATHODE)
- net KeyPadPSU+: now also BJT7.1 (E)
- net LED_B: now also H15.5 (P5), J16.9; no longer R2.1
- net LED_G: now also H15.4 (P4), J16.8; no longer R3.1
- net LED_R: now also H15.7 (P7), J16.7; no longer R1.1
- net Lid_GND: now also H13.4, H2.3; no longer KP1.4 (-), LED1.2 (COMMON_ANODE)
- net Lid_KP_+: now also H13.5; no longer KP1.5 (+)
- net Lid_KP_RX: now also H13.1; no longer KP1.1 (RX)
- net Lid_KP_TX: now also H13.2; no longer KP1.2 (TX)
- net OLED_CS: now also J15.17; no longer U2.J3_17 (GPIO26)
- net OLED_MOSI: now also H16.4, J15.16; no longer U2.J3_16 (GPIO33)
- net OLED_RES: now also J15.14; no longer U2.J3_14 (GPIO35)
- net OLED_SCLK: now also H16.3, J15.22; no longer U2.J3_22 (GPIO47)
- net R+15V: now also H8.3 (P3), H8.4 (P4)
- net R+3V: now also H8.7 (P7), J2.18, J2.2
- net R-15V: now also H8.1 (P1), H8.2 (P2)
- net R-5V: now also H8.6 (P6), J2.10, J2.13, J2.19, J2.26, J2.29, J2.33, J2.40, J2.5
- net R1,9V: now also R1.2, H2.4; no longer H1.1 (P1), LED1.1 (RED_CATHODE)
- net T+15V: now also PS2.22 (+VIN_1), PS2.23 (+VIN_2), IC2.8 (VCC)
- net T+3V: now also DS1.3 (VDD), H7.1 (P1), R4.1, BJT7.3 (C), H16.8, J16.1, J17.2 (Pin_2), S1.2 (COM_1); no longer C1.1
- net T+HEAT: now also J14.5; no longer EC1.9, J14.4, T1.1 (Pin_1)
- net T-15V: now also PS2.2 (-VIN_1), PS2.3 (-VIN_2), IC2.4 (GND)
- net T-3V: now also AST1.2 (-), DS1.1 (GND), H15.6 (P6), H16.6, J15.1, J17.3 (Pin_3); no longer C1.2
- net T-HEAT: now also J14.4; no longer EC1.8, J14.5, T1.2 (Pin_2)
- net T_HEAT_OFF: now also J16.4; no longer U2.J1_4 (GPIO2)
- net T_HEAT_ON: now also J16.3; no longer U2.J1_3 (GPIO1)
- net T_RX: now also IC2.2 (RX); no longer J14.7
- net T_TX: now also IC2.3 (TX); no longer J14.8
- net Tn+15V: now also J1.5, H17.3 (P3), H17.4 (P4); no longer J1.4
- net Tn+3V: now also H17.7 (P7)
- net Tn-15V: now also J1.4, H17.1 (P1), H17.2 (P2); no longer J1.5
- net Tn-5V: now also H17.6 (P6)
- net Tn_RX: now also H18.1 (P1)
- net Tn_TX: now also H18.2 (P2)
- net U1RXD: now also J16.20; no longer U2.J1_20 (GPIO18)
- net U1TXD: now also J16.19; no longer U2.J1_19 (GPIO17)
- removed net 3V3: DS1.3 (VDD), H11.2 (P2), H4.7 (P7), H7.1 (P1), NHD1.2 (VDD), R4.1
- net CS renamed O_CS
- net O_CS: no longer NHD1.15 (CS)
- net D0 renamed O_D0
- net O_D0: no longer NHD1.7 (D0)
- net D1 renamed O_D1
- net O_D1: no longer NHD1.8 (D1)
- net D2 renamed O_D2
- net O_D2: no longer NHD1.9 (D2)
- net DS18B20 renamed T_DS18B20
- net T_DS18B20: now also J16.6
- removed net GND: AST1.2 (-), DS1.1 (GND), H11.1 (P1), H11.10 (P10), H11.11 (P11), H11.12 (P12), H11.13 (P13), H11.14 (P14), H11.17 (P17), H11.18 (P18), H11.19 (P19), H11.20 (P20), H11.3 (P3), H11.4 (P4), H11.5 (P5), H11.6 (P6), H15.6 (P6), H4.6 (P6), NHD1.1 (VSS), NHD1.10 (D3), NHD1.11 (D4), NHD1.12 (D5), NHD1.13 (D6), NHD1.14 (D7), NHD1.17 (BS0), NHD1.18 (BS1), NHD1.19 (BS2), NHD1.20 (VSS(Frame)), NHD1.3 (REGVDD), NHD1.4 (D/C), NHD1.5 (R/W), NHD1.6 (E)
- net OLED_SOMI: no longer names the net of U2.J3_15 (GPIO34)
- net OLED_SOMI: no longer H9.3 (P3)
- net PIEZO renamed T_PIEZO
- net T_PIEZO: now also J16.5
- net RES renamed O_RES
- net O_RES: no longer NHD1.16 (RES)
- net RU+5V renamed R+5V
- net R+5V: now also J2.1, J2.3
- new net: H1.1 (P1), R1.1
- new net: H1.3 (P3), R2.1
- new net: H1.4 (P4), R3.1
- new net: BJT7.2 (B), R5.2
- new net B_BUZ: J17.9 (Pin_9)
- new net B_D+: J17.7 (Pin_7)
- new net B_D-: J17.6 (Pin_6)
- new net B_LED1: J17.10 (Pin_10)
- new net B_LED2: J17.11 (Pin_11)
- new net B_RX: J15.5, J17.4 (Pin_4)
- new net B_TRIG: J15.7, J17.12 (Pin_12), S1.3 (NO_1)
- new net B_TX: J15.6, J17.5 (Pin_5)
- new net E_RST: J15.2, J15.4
- new net OLED_MISO: H16.5, H9.3 (P3), J15.15
- new net O_3V: C1.1, H11.2 (P2), H4.7 (P7)
- new net O_GND: C1.2, H11.1 (P1), H11.10 (P10), H11.11 (P11), H11.12 (P12), H11.13 (P13), H11.14 (P14), H11.17 (P17), H11.18 (P18), H11.19 (P19), H11.20 (P20), H11.3 (P3), H11.4 (P4), H11.5 (P5), H11.6 (P6), H4.6 (P6)
- new net RFID_CS: H16.2, J15.13
- new net RFID_RST: H16.7, J15.12
- new net T2+HEAT: EC1.9, T1.2 (Pin_2)
- new net T2-HEAT: EC1.8, T1.1 (Pin_1)
- new net T_KeyPadON: J16.10, R5.1
- new net T_RY: IC2.6 (RY), J14.7
- new net T_TY: IC2.5 (TY), J14.8
- no-connect marks 22 -> 203
Other:
- note added: "==> FPC cable to 12P FPC breakout board ==>"
- note added: "B_GND"
- note added: "B_VCC"
- note added: "Female header mount for easy maintenance."
- note added: "Plug LED legs to header"
- note added: "RFID board comes with right-angle headers. ==> Push headers to Toveri female header."
- note added: "Remove JST female header and push lid PCB in"
- note added: "USB to PCB ==>"
- note removed: "Has attached USB-cable. Cut it and use the male head to plug to raspberry pi"
- note removed: "KeyPad controller"
- note removed: "Stacking header"
- note removed: "To Raspberry GPIO"
- note removed: "USB tail to turret"
- moved on the sheet: AST1, C1, CAT6, DS1, H1, H7, J14, KP1, LED1, LH1, LHI1, PS2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
